File: docs/kicad/flash6502/CTRL12.kicad_sch (KiCad schematic)
At the start: 3 parts

Commit message: ok, docs
Connections:
- net INST_done: now also CTRL_ROM1.21 (D7); no longer SYNC12.12 (Q7)
- net INST_s_async: now also CTRL_ROM2.14 (D1); no longer CTRL_ROM2.15 (D2)
- net ~{PC_e}: now also CTRL_ROM2.20 (D6); no longer CTRL_ROM2.17 (D3)
- net ~{PC_up_async}: now also CTRL_ROM2.15 (D2); no longer CTRL_ROM2.18 (D4), SYNC12.6 (D4)
- net ~{RAM_e}: now also CTRL_ROM2.19 (D5); no longer CTRL_ROM2.13 (D0)
- net ~{RAM_s_async}: now also CTRL_ROM2.13 (D0); no longer CTRL_ROM2.14 (D1)
- net ~{SP_down_async}: now also CTRL_ROM2.18 (D4); no longer CTRL_ROM2.21 (D7), SYNC12.8 (D6)
- net ~{SP_e}: now also CTRL_ROM2.21 (D7); no longer CTRL_ROM2.19 (D5)
- net ~{SP_s_async}: now also CTRL_ROM2.17 (D3); no longer CTRL_ROM2.20 (D6), SYNC12.7 (D5)
- net at SYNC12.9 (D7): no longer CTRL_ROM1.21 (D7)
- net ~{PC_up}: no longer names the net of SYNC12.15 (Q4)
- net ~{SP_down}: no longer names the net of SYNC12.13 (Q6)
- net ~{SP_s}: no longer names the net of SYNC12.14 (Q5)
- no-connect marks 2 -> 12
Changed lines of the file:
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@@
 (kicad_sch (version 20211123) (generator eeschema)
   (paper "A4")
+  (no_connect (at 97.79 46.99))
   (no_connect (at 160.02 81.28))
+  (no_connect (at 102.87 -8.89))
   (no_connect (at 34.29 82.55))
+  (no_connect (at 123.19 46.99))
+  (no_connect (at 97.79 52.07))
+  (no_connect (at 123.19 54.61))
+  (no_connect (at 97.79 49.53))
+  (no_connect (at 123.19 52.07))
+  (no_connect (at 44.45 -6.35))
+  (no_connect (at 97.79 54.61))
+  (no_connect (at 123.19 49.53))
   (wire (pts (xy 64.77 44.45) (xy 97.79 44.45))
     (stroke (width 0) (type default) (color 0 0 0 0))
   )
-  (wire (pts (xy 64.77 54.61) (xy 97.79 54.61))
-    (stroke (width 0) (type default) (color 0 0 0 0))
-  )
   (wire (pts (xy 64.77 36.83) (xy 97.79 36.83))
     (stroke (width 0) (type default) (color 0 0 0 0))
@@
     (stroke (width 0) (type default) (color 0 0 0 0))
   )
-  (label "~{PC_up_async}" (at 190.5 45.72 0)
-    (effects (font (size 1.27 1.27)) (justify left bottom))
-  )
-  (label "~{SP_s_async}" (at 190.5 50.8 0)
-    (effects (font (size 1.27 1.27)) (justify left bottom))
-  )
-  (label "~{PC_up_async}" (at 97.79 46.99 180)
-    (effects (font (size 1.27 1.27)) (justify right bottom))
-  )
-  (label "~{SP_down_async}" (at 190.5 53.34 0)
-    (effects (font (size 1.27 1.27)) (justify left bottom))
-  )
-  (label "~{SP_down_async}" (at 97.79 52.07 180)
-    (effects (font (size 1.27 1.27)) (justify right bottom))
-  )
-  (label "~{SP_s_async}" (at 97.79 49.53 180)
-    (effects (font (size 1.27 1.27)) (justify right bottom))
-  )
   (global_label "~{CTRL_PC_e}" (shape input) (at 160.02 53.34 180) (fields_autoplaced)
     (effects (font (size 1.27 1.27)) (justify right))
@@
     )
   )
-  (global_label "~{SP_down}" (shape output) (at 123.19 52.07 0) (fields_autoplaced)
-    (effects (font (size 1.27 1.27)) (justify left))
-    (property "Intersheet References" "${INTERSHEET_REFS}" (id 0) (at 133.8279 51.9906 0)
-      (effects (font (size 1.27 1.27)) (justify left) hide)
-    )
-  )
   (global_label "STEP1" (shape input) (at 34.29 39.37 180) (fields_autoplaced)
     (effects (font (size 1.27 1.27)) (justify right))
@@
     )
   )
+  (global_label "~{PC_e}" (shape output) (at 190.5 50.8 0) (fields_autoplaced)
+    (effects (font (size 1.27 1.27)) (justify left))
+    (property "Intersheet References" "${INTERSHEET_REFS}" (id 0) (at 197.5093 50.7206 0)
+      (effects (font (size 1.27 1.27)) (justify left) hide)
+    )
+  )
+  (global_label "~{SP_e}" (shape output) (at 190.5 53.34 0) (fields_autoplaced)
+    (effects (font (size 1.27 1.27)) (justify left))
+    (property "Intersheet References" "${INTERSHEET_REFS}" (id 0) (at 197.4488 53.2606 0)
+      (effects (font (size 1.27 1.27)) (justify left) hide)
+    )
+  )
   (global_label "INST2" (shape input) (at 160.02 66.04 180) (fields_autoplaced)
     (effects (font (size 1.27 1.27)) (justify right))
@@
     )
   )
-  (global_label "~{PC_e}" (shape output) (at 190.5 43.18 0) (fields_autoplaced)
-    (effects (font (size 1.27 1.27)) (justify left))
-    (property "Intersheet References" "${INTERSHEET_REFS}" (id 0) (at 197.5093 43.1006 0)
-      (effects (font (size 1.27 1.27)) (justify left) hide)
-    )
-  )
-  (global_label "~{RAM_s_async}" (shape output) (at 190.5 38.1 0) (fields_autoplaced)
-    (effects (font (size 1.27 1.27)) (justify left))
-    (property "Intersheet References" "${INTERSHEET_REFS}" (id 0) (at 205.0688 38.0206 0)
-      (effects (font (size 1.27 1.27)) (justify left) hide)
-    )
-  )
   (global_label "STEP2" (shape input) (at 160.02 40.64 180) (fields_autoplaced)
     (effects (font (size 1.27 1.27)) (justify right))
@@
     )
   )
-  (global_label "~{PC_up}" (shape output) (at 123.19 46.99 0) (fields_autoplaced)
-    (effects (font (size 1.27 1.27)) (justify left))
-    (property "Intersheet References" "${INTERSHEET_REFS}" (id 0) (at 131.4088 46.9106 0)
+  (global_label "~{RAM_e}" (shape output) (at 190.5 48.26 0) (fields_autoplaced)
+    (effects (font (size 1.27 1.27)) (justify left))
+    (property "Intersheet References" "${INTERSHEET_REFS}" (id 0) (at 198.7793 48.1806 0)
+      (effects (font (size 1.27 1.27)) (justify left) hide)
+    )
+  )
+  (global_label "~{RAM_s_async}" (shape output) (at 190.5 35.56 0) (fields_autoplaced)
+    (effects (font (size 1.27 1.27)) (justify left))
+    (property "Intersheet References" "${INTERSHEET_REFS}" (id 0) (at 205.0688 35.4806 0)
       (effects (font (size 1.27 1.27)) (justify left) hide)
     )
@@
     )
   )
-  (global_label "INST_s_async" (shape output) (at 190.5 40.64 0) (fields_autoplaced)
-    (effects (font (size 1.27 1.27)) (justify left))
-    (property "Intersheet References" "${INTERSHEET_REFS}" (id 0) (at 205.3712 40.5606 0)
-      (effects (font (size 1.27 1.27)) (justify left) hide)
-    )
-  )
   (global_label "INST1" (shape input) (at 34.29 64.77 180) (fields_autoplaced)
     (effects (font (size 1.27 1.27)) (justify right))
@@
     )
   )
+  (global_label "~{SP_s_async}" (shape output) (at 190.5 43.18 0) (fields_autoplaced)
+    (effects (font (size 1.27 1.27)) (justify left))
+    (property "Intersheet References" "${INTERSHEET_REFS}" (id 0) (at 203.7383 43.1006 0)
+      (effects (font (size 1.27 1.27)) (justify left) hide)
+    )
+  )
   (global_label "INST4" (shape input) (at 34.29 72.39 180) (fields_autoplaced)
     (effects (font (size 1.27 1.27)) (justify right))
@@
     )
   )
-  (global_label "INST_done" (shape output) (at 123.19 54.61 0) (fields_autoplaced)
-    (effects (font (size 1.27 1.27)) (justify left))
-    (property "Intersheet References" "${INTERSHEET_REFS}" (id 0) (at 135.2188 54.5306 0)
+  (global_label "~{PC_up_async}" (shape output) (at 190.5 40.64 0) (fields_autoplaced)
+    (effects (font (size 1.27 1.27)) (justify left))
+    (property "Intersheet References" "${INTERSHEET_REFS}" (id 0) (at 205.0688 40.5606 0)
+      (effects (font (size 1.27 1.27)) (justify left) hide)
+    )
+  )
+  (global_label "INST_s_async" (shape output) (at 190.5 38.1 0) (fields_autoplaced)
+    (effects (font (size 1.27 1.27)) (justify left))
+    (property "Intersheet References" "${INTERSHEET_REFS}" (id 0) (at 205.3712 38.0206 0)
       (effects (font (size 1.27 1.27)) (justify left) hide)
     )
@@
     )
   )
-  (global_label "~{RAM_e}" (shape output) (at 190.5 35.56 0) (fields_autoplaced)
-    (effects (font (size 1.27 1.27)) (justify left))
-    (property "Intersheet References" "${INTERSHEET_REFS}" (id 0) (at 198.7793 35.4806 0)
-      (effects (font (size 1.27 1.27)) (justify left) hide)
-    )
-  )
   (global_label "X_s" (shape output) (at 123.19 44.45 0) (fields_autoplaced)
     (effects (font (size 1.27 1.27)) (justify left))
@@
     )
   )
-  (global_label "~{SP_s}" (shape output) (at 123.19 49.53 0) (fields_autoplaced)
-    (effects (font (size 1.27 1.27)) (justify left))
-    (property "Intersheet References" "${INTERSHEET_REFS}" (id 0) (at 130.0783 49.4506 0)
-      (effects (font (size 1.27 1.27)) (justify left) hide)
-    )
-  )
   (global_label "INST7" (shape input) (at 160.02 78.74 180) (fields_autoplaced)
     (effects (font (size 1.27 1.27)) (justify right))
@@
     )
   )
-  (global_label "~{SP_e}" (shape output) (at 190.5 48.26 0) (fields_autoplaced)
-    (effects (font (size 1.27 1.27)) (justify left))
-    (property "Intersheet References" "${INTERSHEET_REFS}" (id 0) (at 197.4488 48.1806 0)
+  (global_label "INST_done" (shape output) (at 64.77 54.61 0) (fields_autoplaced)
+    (effects (font (size 1.27 1.27)) (justify left))
+    (property "Intersheet References" "${INTERSHEET_REFS}" (id 0) (at 76.7988 54.5306 0)
       (effects (font (size 1.27 1.27)) (justify left) hide)
     )
@@
       (effects (font (size 1.27 1.27)) (justify left) hide)
     )
+  )
+  (global_label "~{SP_down_async}" (shape output) (at 190.5 45.72 0) (fields_autoplaced)
+    (effects (font (size 1.27 1.27)) (justify left))
+    (property "Intersheet References" "${INTERSHEET_REFS}" (id 0) (at 207.4879 45.6406 0)
+      (effects (font (size 1.27 1.27)) (justify left) hide)
+    )
