File: docs/kicad/flash6502/CTRL45.kicad_sch (KiCad schematic)
At the start: 3 parts

Commit message: kicad update
Parts:
- added LEDI0, LEDI1, LEDI2, LEDI3, LEDI4, LEDI5, LEDI6, LEDI7: LED, symbol Device:LED
- added RLI0, RLI1, RLI2, RLI3, RLI4, RLI5, RLI6, RLI7: 1k, symbol Device:R
Connections:
- net GND: now also RLI0.2, RLI1.2, RLI2.2, RLI3.2, RLI4.2, RLI5.2, RLI6.2, RLI7.2
- net INST0: now also LEDI0.2 (A)
- net INST1: now also LEDI1.2 (A)
- net INST2: now also LEDI2.2 (A)
- net INST3: now also LEDI3.2 (A)
- net INST4: now also LEDI4.2 (A)
- net INST5: now also LEDI5.2 (A)
- net INST6: now also LEDI6.2 (A)
- net INST7: now also LEDI7.2 (A)
- new net: LEDI6.1 (K), RLI6.1
- new net: LEDI3.1 (K), RLI3.1
- new net: LEDI2.1 (K), RLI2.1
- new net: LEDI7.1 (K), RLI7.1
- new net: LEDI4.1 (K), RLI4.1
- new net: LEDI1.1 (K), RLI1.1
- new net: LEDI0.1 (K), RLI0.1
- new net: LEDI5.1 (K), RLI5.1
Other:
- note removed: "TODO: Add INST LEDS"

Commit message: ok, docs
Connections:
- net EAL_s_async: now also CTRL_ROM4.17 (D3); no longer CTRL_ROM4.15 (D2)
- net ~{PCL_s_async}: now also CTRL_ROM4.15 (D2); no longer CTRL_ROM4.17 (D3)
Changed lines of the file:
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@@
     (stroke (width 0) (type default) (color 0 0 0 0))
+  )
+  (label "EAL_s_async" (at 115.57 44.45 0)
+    (effects (font (size 1.27 1.27)) (justify left bottom))
   )
   (label "~{PCH_s_async}" (at 223.52 39.37 180)
@@
     (effects (font (size 1.27 1.27)) (justify right bottom))
   )
+  (label "~{PCL_s_async}" (at 115.57 41.91 0)
+    (effects (font (size 1.27 1.27)) (justify left bottom))
+  )
   (label "EAL_s_async" (at 223.52 44.45 180)
     (effects (font (size 1.27 1.27)) (justify right bottom))
@@
   )
   (label "EAH_s_async" (at 115.57 39.37 0)
-    (effects (font (size 1.27 1.27)) (justify left bottom))
-  )
-  (label "EAL_s_async" (at 115.57 41.91 0)
-    (effects (font (size 1.27 1.27)) (justify left bottom))
-  )
-  (label "~{PCL_s_async}" (at 115.57 44.45 0)
     (effects (font (size 1.27 1.27)) (justify left bottom))
   )
@@
   (symbol (lib_id "power:GND") (at 36.83 36.83 270) (unit 1)
     (in_bom yes) (on_board yes) (fields_autoplaced)
-    (property "Reference" "#PWR?" (id 0) (at 30.48 36.83 0)
+    (property "Reference" "#PWR0313" (id 0) (at 30.48 36.83 0)
       (effects (font (size 1.27 1.27)) hide)
     )
@@
   (symbol (lib_id "power:GND") (at 36.83 111.76 270) (unit 1)
     (in_bom yes) (on_board yes)
-    (property "Reference" "#PWR?" (id 0) (at 30.48 111.76 0)
+    (property "Reference" "#PWR0311" (id 0) (at 30.48 111.76 0)
       (effects (font (size 1.27 1.27)) hide)
     )
@@
   (symbol (lib_id "power:GND") (at 36.83 57.15 270) (unit 1)
     (in_bom yes) (on_board yes) (fields_autoplaced)
-    (property "Reference" "#PWR?" (id 0) (at 30.48 57.15 0)
+    (property "Reference" "#PWR0309" (id 0) (at 30.48 57.15 0)
       (effects (font (size 1.27 1.27)) hide)
     )
@@
   (symbol (lib_id "power:GND") (at 36.83 46.99 270) (unit 1)
     (in_bom yes) (on_board yes) (fields_autoplaced)
-    (property "Reference" "#PWR?" (id 0) (at 30.48 46.99 0)
+    (property "Reference" "#PWR0314" (id 0) (at 30.48 46.99 0)
       (effects (font (size 1.27 1.27)) hide)
     )
@@
   (symbol (lib_id "power:GND") (at 36.83 77.47 270) (unit 1)
     (in_bom yes) (on_board yes)
-    (property "Reference" "#PWR?" (id 0) (at 30.48 77.47 0)
+    (property "Reference" "#PWR0233" (id 0) (at 30.48 77.47 0)
       (effects (font (size 1.27 1.27)) hide)
     )
@@
   (symbol (lib_id "power:GND") (at 36.83 100.33 270) (unit 1)
     (in_bom yes) (on_board yes)
-    (property "Reference" "#PWR?" (id 0) (at 30.48 100.33 0)
+    (property "Reference" "#PWR0312" (id 0) (at 30.48 100.33 0)
       (effects (font (size 1.27 1.27)) hide)
     )
@@
   (symbol (lib_id "power:GND") (at 36.83 67.31 270) (unit 1)
     (in_bom yes) (on_board yes) (fields_autoplaced)
-    (property "Reference" "#PWR?" (id 0) (at 30.48 67.31 0)
+    (property "Reference" "#PWR0310" (id 0) (at 30.48 67.31 0)
       (effects (font (size 1.27 1.27)) hide)
     )
@@
   (symbol (lib_id "power:GND") (at 36.83 88.9 270) (unit 1)
     (in_bom yes) (on_board yes)
-    (property "Reference" "#PWR?" (id 0) (at 30.48 88.9 0)
-      (effects (font (size 1.27 1.27)) hide)
-    )
+    (property "Reference" "#PWR0308" (id 0) (at 30.48 88.9 0)
+      (effects (font (size 1.27 1.27)) hide)
+    )
