File: docs/kicad/flash6502/RAM.kicad_sch (KiCad schematic)
At the start: 6 parts

Commit message: ok, docs
Parts:
- removed INST: 74HC373, symbol 74xx:74HC373
- added INST: 74HC574, symbol 74xx:74HCT574
Connections:
- net +5V: now also INST.20 (VCC)
- net D0: now also INST.2 (D0)
- net D1: now also INST.3 (D1)
- net D2: now also INST.4 (D2)
- net D3: now also INST.5 (D3)
- net D4: now also INST.6 (D4)
- net D5: now also INST.7 (D5)
- net D6: now also INST.8 (D6)
- net D7: now also INST.9 (D7)
- net GND: now also INST.1 (OE), INST.10 (GND)
- net INST0: now also INST.19 (Q0)
- net INST1: now also INST.18 (Q1)
- net INST2: now also INST.17 (Q2)
- net INST3: now also INST.16 (Q3)
- net INST4: now also INST.15 (Q4)
- net INST5: now also INST.14 (Q5)
- net INST6: now also INST.13 (Q6)
- net INST7: now also INST.12 (Q7)
- net INST_s: now also INST.11 (Cp)
