File: docs/kicad/flash6502/Status.kicad_sch (KiCad schematic)
At the start: 21 parts

Commit message: ok
Other:
- note added: "Pull-down resistors for ALU flags"
- note removed: "TODO: These are not hooked-up on the board!"
Changed lines of the file:
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@@
     (stroke (width 0) (type default) (color 0 0 0 0))
   )
-  (text "TODO: These are not hooked-up on the board!" (at 31.75 100.33 0)
+  (text "Pull-down resistors for ALU flags" (at 31.75 100.33 0)
     (effects (font (size 1.27 1.27)) (justify left bottom))
   )
