File: docs/kicad/flash6502/ALU.kicad_sch (KiCad schematic)
At the start: 4 parts

Commit message: ok
Other:
- note removed: "TODO: ALU_L_* local labels don't have pull-down resistors!"
Changed lines of the file:
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@@
   (no_connect (at 185.42 54.61))
   (no_connect (at 154.94 82.55))
-  (text "TODO: ALU_L_* local labels don't have pull-down resistors!"
-    (at 143.51 22.86 0)
-    (effects (font (size 1.27 1.27)) (justify left bottom))
-  )
   (label "A5" (at 100.33 67.31 180)
     (effects (font (size 1.27 1.27)) (justify right bottom))
